Commit message: fix: add prefix to grasp link

File: za6_tools/urdf/none_macro.xacro (robot description, xacro)
@@ -4,5 +4,5 @@
     <!-- URDF for *no* gripper: define grasp_link with no geometry &
          connect it at flange -->
-    <link name="grasp_link"/>
+    <link name="${prefix}grasp_link"/>
     <!-- joint list -->
     <joint name="${prefix}grasp_joint" type="fixed">

File: za6_tools/urdf/pivot_gripper_macro.xacro (robot description, xacro)
@@ -126,8 +126,8 @@
     </joint>
     <!-- Attach grasp_link to gripper base for now -->
-    <link name="grasp_link" />
-    <joint name="grasp_joint" type="fixed">
-      <parent link="$(arg prefix)pivot_gripper_base" />
-      <child link="grasp_link" />
+    <link name="${prefix}grasp_link" />
+    <joint name="${prefix}grasp_joint" type="fixed">
+    <parent link="${prefix}pivot_gripper_base" />
+      <child link="${prefix}grasp_link" />
       <origin xyz="0.0 0.0 0.0" rpy="0.0 0.0 0.0" />
     </joint>

File: za6_tools/urdf/robotiq_hand_e_macro.xacro (robot description, xacro)
@@ -79,8 +79,8 @@
     </joint>
     <!-- Attach grasp_link to gripper body for now -->
-    <link name="grasp_link" />
-    <joint name="grasp_joint" type="fixed">
+    <link name="${prefix}grasp_link" />
+    <joint name="${prefix}grasp_joint" type="fixed">
       <parent link="${prefix}hand_e_body" />
-      <child link="grasp_link" />
+      <child link="${prefix}grasp_link" />
       <origin xyz="0.0 0.0 0.135" rpy="0.0 0.0 0.0" />
     </joint>

File: za6_tools/urdf/versabuilt_multigrip_macro.xacro (robot description, xacro)
@@ -67,8 +67,8 @@
     </joint>
     <!-- Attach grasp_link to multigrip base for now -->
-    <link name="grasp_link" />
-    <joint name="grasp_joint" type="fixed">
-      <parent link="$(arg prefix)multigrip_base_and_fixed_jaw" />
-      <child link="grasp_link" />
+    <link name="${prefix}grasp_link" />
+    <joint name="${prefix}grasp_joint" type="fixed">
+      <parent link="${prefix}multigrip_base_and_fixed_jaw" />
+      <child link="${prefix}grasp_link" />
       <origin xyz="0.0 0.0 0.0" rpy="0.0 0.0 0.0" />
     </joint>
